File: Power/power.sch (EAGLE design)
At the start: 93 parts, among them IC1 LM317MSTT3, IC2 LM317MSTT3, IC3 LM317MSTT3, IC4 LM317MSTT3, IC5 AD8610ARZR-8, IC6 AD8610ARZR-8, X1 STEREOJACK, X2 STEREOJACK

Commit message: Created Modular branch
This commit splits the power supply from the amp itself.
Parts:
- removed C13, C22, C26, C9: 470uF/35V, rcl:CPOL-USE5-13
- removed C33, C34, C36, C37, C38, C39, C40: 100nF/50V, rcl:C-USC0805
- removed C35: 100pF/100V, rcl:C-USC0805
- removed IC5, IC6: AD8610ARZR-8, ad8610arz:AD8610ARZR-8
- removed R15, R18, R19, R20, R21, R25, R26, R27, R30, R31, R32, R33, R34, R36: 1k0, rcl:R-US_M0805
- removed R16, R17, R28, R29: 470k, rcl:R-US_M0805
- removed R22, R35: 10, rcl:R-US_M0805
- removed R23, R24, R37, R38: 220, rcl:R-US_M0805
- removed S1, S2: (no value), adafruit:EG1218S
- removed U$3: TPA6120, tpa6120:TPA6120
- removed X1, X2: STEREOJACK, adafruit:STEREOJACK
- C27, C29, C30: value 100nF/50V -> 470uF/35V; device rcl:C-USC0805 -> rcl:CPOL-USE5-13
- C28: value 100pF/100V -> 470uF/35V; device rcl:C-USC0805 -> rcl:CPOL-USE5-13
- C31, C32: value 100nF/50V -> 2200uF/35V; device rcl:C-USC0805 -> rcl:CPOL-USE5-13
- IC3, IC4: value LM317MSTT3 -> LM337IMP; device v-reg:LM317MSTT3 -> AWJLEagleLib:LM337IMP
Connections:
- removed net HP_IN_L: C27.1, R16.1, X1.2
- removed net HP_IN_R: C34.1, R28.1, X1.5
- removed net N$10: C28.1, IC5.+IN, R15.1
- removed net N$12: IC5.-IN, R18.1, R19.2
- removed net N$13: IC5.OUT, R19.1, R20.2
- removed net N$15: R21.2, R22.2, U$3.LOUT
- removed net N$16: C33.1, R25.1, R26.1, U$3.LIN+
- removed net N$18: R22.1, R23.2, R24.2, S1.P
- removed net N$19: R23.1, R24.1, S1.S, X2.2
- removed net N$20: R33.1, R35.2, U$3.ROUT
- removed net N$21: C34.2, R27.2, R29.1
- removed net N$22: C35.1, IC6.+IN, R27.1
- removed net N$23: IC6.-IN, R30.1, R31.2
- removed net N$24: IC6.OUT, R31.1, R32.2
- removed net N$25: R32.1, R33.2, U$3.RIN-
- removed net N$26: R35.1, R37.2, R38.2, S2.P
- removed net N$27: C40.1, R34.2, R36.2, U$3.RIN+
- removed net N$28: R37.1, R38.1, S2.S, X2.5
- removed net N$3: B1.+, C1.1, C10.1, C3.1, C5.1, C6.+, IC1.IN, IC2.IN, R1.2
- removed net N$5: R20.1, R21.1, U$3.LIN-
- removed net N$6: C27.2, R15.2, R17.1
- removed net N$9: B2.-, C14.1, C16.1, C18.-, C19.1, C23.1, IC3.IN, IC4.IN, R8.2
- new net +VSS_NOREG: B1.+, C1.1, C10.1, C3.1, C31.+, C5.1, C6.+, IC1.IN, IC2.IN, R1.2
- new net -VSS_NOREG: B2.-, C14.1, C16.1, C18.-, C19.1, C23.1, C32.-, IC3.IN, IC3.P$1, IC4.IN, IC4.P$1, R8.2
- net +12V_L: now also C27.+; no longer C30.1, C31.1, C9.+, IC5.V+, U$3.LVCC+
- net +12V_R: now also C28.+; no longer C13.+, C37.1, C38.1, IC6.V+, U$3.RVCC+
- net -12V_L: now also C29.-; no longer C22.+, C29.1, C32.1, IC5.V-, U$3.LVCC-
- net -12V_R: now also C30.-; no longer C26.+, C36.1, C39.1, IC6.V-, U$3.RVCC-
- net GND: now also C27.-, C28.-, C29.+, C30.+, C31.-, C32.+; no longer C13.-, C22.-, C26.-, C28.2, C29.2, C30.2, C31.2, C32.2, C33.2, C35.2, C36.2, C37.2, C38.2, C39.2, C40.2, C9.-, R16.2, R17.2, R18.2, R25.2, R26.2, R28.2, R29.2, R30.2, R34.1, R36.1, U$3.NC1, U$3.NC10, U$3.NC2, U$3.NC3, U$3.NC4, U$3.NC5, U$3.NC6, U$3.NC7, U$3.NC8, U$3.NC9, U$3.THERM, X1.1, X2.1
Other:
- note added: "1"
- note added: "2"
- note added: "3"
- note added: "4"
- note removed: "** CHANGE TO LM337 **"
- moved on the sheet: C10, C11, C12, C19, C20, C21, C23, C24, C25, C5, C7, C8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
