File: Amp/tpa6120-v1_0_0_0-optim.sch (EAGLE design)
At the start: 42 parts, among them IC7 AD8610ARZR-8, IC8 AD8610ARZR-8, X1 STEREOJACK

Commit message: Optimized with 2-channel op-amp
Optimized with 2-channel op-amp
Parts:
- removed C43, C44: 100nF/50V, rcl:C-USC0805
- removed IC7, IC8: AD8610ARZR-8, ad8610arz:AD8610ARZR-8
- added IC1: AD8620R, analog-devices:AD8620R
- added U$2: (no value), audio-pots:ALPS_BLUE
- added X2: STEREOJACK, adafruit:STEREOJACK
- C10, C5, C6, C7, C8, C9: device rcl:C-USC0805 -> rcl:C-USC0402
- C42, C49, C50, C51: device rcl:C-USC0805 -> rc-master-smd:C_0603
- R1, R10, R2, R3, R4, R5, R6, R7, R8, R9: device rcl:R-US_M0805 -> rcl:R-US_R0402
- R39, R40, R41, R42, R43, R51, R52, R53, R54, R55: device rcl:R-US_M0805 -> rc-master-smd:R_0603
Connections:
- new net N$23: R6.1, X2.5
- new net N$24: R5.1, X2.2
- new net POT_L: C41.1, R40.1, U$2G$1.2
- new net POT_R: C48.1, R52.1, U$2G$2.2
- net +12V_L: no longer C44.1, IC7.V+
- net +12V_R: now also IC1P.V+; no longer IC8.V+
- net -12V_L: now also C3.-; no longer C3.+, C43.1, IC7.V-
- net -12V_R: now also C4.-, IC1P.V-; no longer C4.+, IC8.V-
- net BUFF_L_OUT: now also IC1A.OUT; no longer IC7.OUT
- net BUFF_R_OUT: now also IC1B.OUT; no longer IC8.OUT
- net GND: now also C3.+, C4.+, U$2G$1.3, U$2G$2.3, X2.1; no longer C3.-, C4.-, C43.2, C44.2
- net HP_IN_L: now also U$2G$1.1, X1.3; no longer C41.1, R40.1
- net HP_IN_R: now also U$2G$2.1, X1.4; no longer C48.1, R52.1
- net N$31: now also IC1A.IN+; no longer IC7.+IN
- net N$32: now also IC1A.IN-; no longer IC7.-IN
- net N$40: now also IC1B.IN+; no longer IC8.+IN
- net N$41: now also IC1B.IN-; no longer IC8.-IN
Other:
- note added: "- Board requires 2 +/-12V Power Supplies"
- note added: "- Can use any precision op amp"
- note added: "- TPA6120 Based"
- note added: "- This design uses an AD8620 as"
- note added: "1.0.0.0-OPT"
- note added: "4/9/2014"
- note added: "Amp Section"
- note added: "Audio IN"
- note added: "Op Amp Power"
- note added: "Power Entry"
- note added: "TPA6120 Headphone Amp"
- note added: "Travis Estep"
- note added: "Version 1.0.0.0-opt"
- note added: "opposed to 2 single AD8610s"
- moved on the sheet: C1, C2, C3, C4, C41, C42, C48, C49, C50, C51, R39, R40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
